Commit message: Work done to get visualization moving in x and y. Possible issue with the dynamics.

File: julia/zoe2.urdf (robot description, URDF)
Before this commit: robot zoe2, 10 links, 9 joints
Links:
- link back_axle: geometry collision box size=1.5899999999999999 0.1 0.1; visual mesh filename=meshes/front_axle.obj
- link back_roll: geometry collision box size=0.1 0.1 0.4; visual mesh filename=meshes/back_hinge.obj
- link chassis: geometry collision box size=1.2 1.5 0.5; visual mesh filename=meshes/chassis.obj
- link front_axle: geometry collision box size=1.5899999999999999 0.1 0.1; visual mesh filename=meshes/front_axle.obj
- link front_roll: geometry collision box size=0.1 0.1 0.4; visual mesh filename=meshes/back_hinge.obj
- link wheel_back_left: geometry collision cylinder length=0.05 radius=0.325; visual mesh filename=meshes/wheel_back_right.obj
- link wheel_back_right: geometry collision cylinder length=0.05 radius=0.325; visual mesh filename=meshes/wheel_back_right.obj
- link wheel_front_left: geometry collision cylinder length=0.05 radius=0.325; visual mesh filename=meshes/wheel_back_right.obj
- link wheel_front_right: geometry collision cylinder length=0.05 radius=0.325; visual mesh filename=meshes/wheel_back_right.obj
